File: db19-to-idc20/db19-to-idc20.kicad_pcb (KiCad board)
At the start: 2 copper layers, 41 x 20.6 mm, 6 parts, among them J1 DB19_Plug, J2 IDC-20

Commit message: Add Combo version
Other:
- board text removed: "SmartPortSD SMD v1.1 github.com/djtersteegc/smartportsd-smd PCB by Chris Tersteeg"
Changed lines of the file:
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@@
   (gr_arc (start 173.355 111.76) (mid 174.702038 112.317962) (end 175.26 113.665)
     (stroke (width 0.1) (type default)) (layer "Edge.Cuts"))
-  (gr_text "SmartPortSD SMD v1.1\ngithub.com/djtersteegc/smartportsd-smd\nPCB by Chris Tersteeg" (at 154.051 92.075) (layer "B.SilkS")
-    (effects (font (size 1 1) (thickness 0.15)) (justify mirror))
-  )
   (gr_text "2" (at 168.656 119.126) (layer "B.SilkS")
     (effects (font (size 1 1) (thickness 0.15)) (justify left bottom mirror))
@@
     (effects (font (size 1 1) (thickness 0.15)) (justify left bottom))
   )
+  (dimension (type aligned) (layer "B.Cu")
+    (pts (xy 173.355 111.76) (xy 173.358091 132.330395))
+    (height -15.24253)
+    (gr_text "20.5704 mm" (at 190.399076 122.042637 270.0086123) (layer "B.Cu")
+      (effects (font (size 1.5 1.5) (thickness 0.3)))
+    )
+    (format (prefix "") (suffix "") (units 3) (units_format 1) (precision 4))
+    (style (thickness 0.2) (arrow_length 1.27) (text_position_mode 0) (extension_height 0.58642) (extension_offset 0.5) keep_text_aligned)
+  )
+  (dimension (type aligned) (layer "B.Cu")
+    (pts (xy 134.286139 130.425395) (xy 175.263091 130.425395))
+    (height 14.532405)
+    (gr_text "40.9770 mm" (at 154.774615 143.1578) (layer "B.Cu")
+      (effects (font (size 1.5 1.5) (thickness 0.3)))
+    )
+    (format (prefix "") (suffix "") (units 3) (units_format 1) (precision 4))
+    (style (thickness 0.2) (arrow_length 1.27) (text_position_mode 0) (extension_height 0.58642) (extension_offset 0.5) keep_text_aligned)
+  )
   (segment (start 154.051 126.187) (end 154.051 120.015) (width 0.25) (layer "B.Cu") (net 1))
